File: ESP32.sch (KiCad schematic (older format))
At the start: 24 parts

Commit message: actual
Parts:
- added R41: 10k, symbol Device:R
- gave numbers to parts that had none: 24
Connections:
- wire segments 107 -> 110
