File: INL8_v3.sch (KiCad schematic (older format))
At the start: 14 parts

Commit message: actual
Parts:
- removed R?: R, symbol Device:R
- gave numbers to parts that had none: 13
Connections:
- net labels added: 0V, 12V, 12VDC, 5VDC
- wire segments 150 -> 154
Other:
- note added: "EXTERNAL SUPPLY"
